File: pcb/FPGA_MSXtR_TangNano20Kx2/FPGA_MSXtR_TangNano20Kx2.kicad_sch (KiCad schematic)
At the start: 29 parts, among them J1 I/O Expander, J2 Conn_01x06, J3 PICO_GPIO, SW1 SW_SPDT, SW2 SW_SPDT, U5 W25Q32JVSS, U6 W25Q32JVSS

Commit message: FPGA MSXtR TangNano20K 2個バージョン (動作未確認) の PCBデータ
Parts:
- C2, C4, C5: LCSC (none) -> C1525
- C3: LCSC (none) -> C1548
- D1: LCSC (none) -> C2293
- R1: LCSC (none) -> C12246
- R10, R11, R4, R5, R6, R7, R8, R9: LCSC (none) -> C25900
- R2, R3: LCSC (none) -> C25905
- U3: LCSC (none) -> C252335
- U5, U6: LCSC (none) -> C82344
