File: pcb/FPGA_MSXtR_Stack_V9968/StackV9968.kicad_pcb (KiCad board)
At the start: 2 copper layers, 95 x 95 mm, 15 parts, among them J1 MSX_EXBUS_A, J2 MSX_EXBUS_B

Commit message: Updated
Parts:
- renumbered U1 to U2
Connections:
- net 3V3_VDP renamed VDP_3V3
- J1 pad 10: unconnected-(J1-Pin_10-Pad10) -> I2S_DIN
- J1 pad 12: unconnected-(J1-Pin_12-Pad12) -> I2S_EN
- J1 pad 14: unconnected-(J1-Pin_14-Pad14) -> I2S_LRCK
- J1 pad 8: unconnected-(J1-Pin_8-Pad8) -> I2S_BCLK
- J2 pad 5: unconnected-(J2-Pin_5-Pad5) -> SLOT_DATA_DIR
- J2 pad 7: unconnected-(J2-Pin_7-Pad7) -> SLOT_OE_N
- U2 pad 16: SLOT_OE_N -> unconnected-(U2-IOL51B(20)-Pad16)
- U2 pad 17: SLOT_DATA_DIR -> unconnected-(U2-IOL51A(19)-Pad17)
- U2 pad 30: unconnected-(U2-IOR36B(55)-Pad30) -> I2S_LRCK
- U2 pad 32: unconnected-(U2-IOR45A(51)-Pad32) -> I2S_EN
- U2 pad 33: unconnected-(U2-IOR38A(54)-Pad33) -> I2S_DIN
- U2 pad 34: unconnected-(U2-IOR36A(56)-Pad34) -> I2S_BCLK
Routing:
- net I2S_LRCK: track 0.00 -> 85.7 mm
- net I2S_EN: track 0.00 -> 74.2 mm, vias 0 -> 3
- net I2S_DIN: track 0.00 -> 71.8 mm, vias 0 -> 3
- net I2S_BCLK: track 0.00 -> 71.6 mm, vias 0 -> 2
