File: pcb/FPGA_MSXtR_Stack_V9968/StackV9968.kicad_sch (KiCad schematic)
At the start: 9 parts, among them J1 MSX_EXBUS_A, J2 MSX_EXBUS_B

Commit message: Updated
Parts:
- SW1, SW2: symbol My_Symbols:Switch -> My Parts:Switch
- U1: symbol My_Symbols:CLOCK -> My Parts:CLOCK
- U2: symbol My_Symbols:TangNano20K -> My Parts:TangNano20K
Connections:
- net SLOT_GND is gone; now on net GND: J1.36 (Pin_36), J2.37 (Pin_37), J2.40 (Pin_40)
- net SLOT_INT is gone; now on net SLOT_INT_N: U2.23 (IOT44A(71))
- net SLOT_WAIT is gone; now on net SLOT_WAIT_N: U2.24 (IOT40B(72))
- net 3V3: no longer C2.1, SW1.1, SW2.1, U1.4 (3V3), U2.19 (3V3), U2.25 (3V3)
- net SLOT_DATA_DIR: now also J2.5 (Pin_5); no longer U2.17 (IOL51A(19))
- net SLOT_OE_N: now also J2.7 (Pin_7); no longer U2.16 (IOL51B(20))
- net I2S_DIN: now reaches J1.10 (Pin_10)
- net I2S_DIN: now also U2.33 (IOR38A(54))
- net I2S_EN: now reaches J1.12 (Pin_12)
- net I2S_EN: now also U2.32 (IOR45A(51))
- net I2S_LRCK: now reaches J1.14 (Pin_14)
- net I2S_LRCK: now also U2.30 (IOR36B(55))
- net I2S_BCLK: now reaches J1.8 (Pin_8)
- net I2S_BCLK: now also U2.34 (IOR36A(56))
- new net VDP_3V3: C2.1, SW1.1, SW2.1, U1.4 (3V3), U2.19 (3V3), U2.25 (3V3)
- no-connect marks 37 -> 51
