File: pcb/FPGA_MSXtR_Stack_Y8960/StackY8960.kicad_pcb (KiCad board)
At the start: 2 copper layers, 95.2 x 65.4 mm, 61 parts, among them J1 I2S_CONN, J2 SOUNDIN, J3 Conn_02x06_Odd_Even, J4 GND, Q1 NMOS, Q2 NMOS, Q3 NMOS

Commit message: Updated
Parts:
- removed C10, C11, C12, C5, C6, C7, C8, C9: 0.1uF, Capacitor_SMD:C_0402_1005Metric
- removed G1: LOGO, 0-My_Parts:msx_logo_15x5p8
- removed G2: LOGO, 0-My_Parts:usa_10x7
- removed Q1, Q2, Q3: NMOS, 0-My_Parts:MOSFET(SMD)
- removed R1, R2, R3, R4, R5, R6, R7, R8: 4.7k, Resistor_SMD:R_0805_2012Metric
- removed R19, R21: 3.3k, Resistor_SMD:R_0805_2012Metric
- removed R20: 10k, Resistor_SMD:R_0805_2012Metric
- removed U5, U6, U7: ~, Package_SO:SSOP-24_5.3x8.2mm_P0.65mm
- removed U8: ~, 0-My_Parts:QSPI-SRAM 4Mbit (8SOIC)
- removed U9: ~, 0-My_Parts:TangPrimer25K(LOWER)
- added J5: GND, Connector_PinHeader_2.54mm:PinHeader_1x01_P2.54mm_Vertical, F.Cu at (33.5, 63.6)
- added J6: SOUNDIN, Connector_PinHeader_2.54mm:PinHeader_1x01_P2.54mm_Vertical, F.Cu at (33.5, 68.2)
- added REF**: BF@MountingHole_3.2mm_M3, 0-My_Parts:BF@MountingHole_3.2mm_M3, F.Cu at (172.8, 118.6)
- added REF**: BF@MountingHole_3.2mm_M3, 0-My_Parts:BF@MountingHole_3.2mm_M3, F.Cu at (87.8, 33.6)
- added REF**: BF@MountingHole_3.2mm_M3, 0-My_Parts:BF@MountingHole_3.2mm_M3, F.Cu at (87.8, 118.6)
- added REF**: BF@MountingHole_3.2mm_M3, 0-My_Parts:BF@MountingHole_3.2mm_M3, F.Cu at (172.8, 33.6)
- C2: value 15pF -> 0.1uF; footprint Capacitor_SMD:C_0805_2012Metric -> Capacitor_SMD:C_0402_1005Metric
- C3: value 0.1uF -> 15pF; footprint Capacitor_SMD:C_0402_1005Metric -> Capacitor_SMD:C_0805_2012Metric
- J1: value I2S_CONN -> MSX_EXBUS_A; footprint Connector_PinHeader_2.54mm:PinHeader_1x06_P2.54mm_Vertical -> Connector_PinHeader_2.54mm:PinHeader_2x20_P2.54mm_Vertical
- J2: value SOUNDIN -> MSX_EXBUS_B; footprint Connector_PinHeader_2.54mm:PinHeader_1x01_P2.54mm_Vertical -> Connector_PinHeader_2.54mm:PinHeader_2x20_P2.54mm_Vertical
- J3: value Conn_02x06_Odd_Even -> I2S_CONN; footprint Connector_PinSocket_2.54mm:PinSocket_2x06_P2.54mm_Vertical -> Connector_PinHeader_2.54mm:PinHeader_1x06_P2.54mm_Vertical
- J4: value GND -> Conn_02x06_Odd_Even; footprint Connector_PinHeader_2.54mm:PinHeader_1x01_P2.54mm_Vertical -> Connector_PinSocket_2.54mm:PinSocket_2x06_P2.54mm_Vertical
- SW1, SW2: footprint 0-My_Parts:SlideSwitch -> 0-My_Parts:SlideSW_Side
- U1: footprint 0-My_Parts:TangPrimer25K(UPPER) -> My Parts:TangPrimer25K(UPPER)
- U2: footprint 0-My_Parts:MSX Cartridge_1 -> My Parts:TangPrimer25K(LOWER)
- U3: footprint 0-My_Parts:CLOCK -> My Parts:QSPI-SRAM 4Mbit (8SOIC)
- U4: footprint Package_SO:SSOP-24_5.3x8.2mm_P0.65mm -> My Parts:CLOCK
- moved R13 114.8 mm to (20.2, 74.6)
- moved R14 111.6 mm to (24.6, 62.8)
- moved R15 107.2 mm to (24.6, 65.8), turned to 0 degrees
- moved R16 107.0 mm to (24.6, 68.7), turned to 0 degrees
- moved R17 106.9 mm to (24.6, 71.7)
- moved R18 106.8 mm to (24.6, 74.6)
- moved U1 96.7 mm to (29.9, 33.0), turned to 0 degrees
- moved J3 94.2 mm to (58.4, 53.9)
- moved C3 93.8 mm to (38.0, 67.1), turned to 0 degrees
- moved SW2 89.9 mm to (61.7, 49.0), turned to 0 degrees
- moved U2 89.1 mm to (29.9, 51.9)
- moved J1 71.8 mm to (44.1, 25.9), turned to 0 degrees
- moved R12 71.4 mm to (20.2, 71.7), turned to 0 degrees
- moved R11 70.2 mm to (20.2, 68.7), turned to 0 degrees
- moved R10 69.3 mm to (20.2, 65.8), turned to 0 degrees
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Connections:
- C2 pad 1: CLK28M -> +3V3
- C3 pad 1: +3V3 -> CLK28M
- C4 pad 1: +5V -> 5V
- J1 pad 1: AUDIO_MCLK -> SLOT_CS2_N
- J1 pad 2: AUDIO_BCLK -> SLOT_RFSH_N
- J1 pad 3: AUDIO_SDATA -> SLOT_SLTSL1_N
- J1 pad 4: AUDIO_LRCLK -> SLOT_SLTSL0_N
- J1 pad 5: GND -> SLOT_SLTSL2_N
- J1 pad 6: +3V3 -> SLOT_SLTSL3_N
- J2 pad 1: Net-(J2-Pin_1) -> SLOT_SNDIN
- J3 pad 1: GND -> AUDIO_MCLK
- J3 pad 2: GND -> AUDIO_BCLK
- J3 pad 3: unconnected-(J3-Pin_3-Pad3) -> AUDIO_SDATA
- J3 pad 4: +5V -> AUDIO_LRCLK
- J3 pad 5: UART_RX -> GND
- J3 pad 6: JTAG_TCK -> +3V3
- U1 pad 52: +5V -> 5V
- U1 pad 54: +5V -> 5V
- U1 pad 56: +5V -> 5V
- U1 pad 58: +5V -> 5V
- U1 pad 60: +5V -> 5V
- U3 pad 1: +3V3 -> SRAM_CS_N
- U3 pad 2: GND -> SRAM_SIO1
- U3 pad 3: CLK28M -> SRAM_SIO2
- U3 pad 4: +3V3 -> GND
- U4 pad 2: SLOT_BUSDIR -> GND
- U4 pad 3: SLOT_D7 -> CLK28M
- U4 pad 4: SLOT_D6 -> +3V3
Routing:
- net GND: track 415.5 -> 0.00 mm, vias 117 -> 0
- net +3V3: track 302.4 -> 0.00 mm, vias 9 -> 0
- net +5V: track 215.3 -> 0.00 mm, vias 8 -> 0
- net SLOT_SLTSL_N: track 66.3 -> 0.00 mm, vias 4 -> 0
- net Net-(J2-Pin_1): track 64.8 -> 0.00 mm, vias 1 -> 0
- net SLOT_IORQ_N: track 64.3 -> 0.00 mm, vias 4 -> 0
- net SLOT_MERQ_N: track 62.7 -> 0.00 mm, vias 4 -> 0
- net SLOT_INTR: track 55.5 -> 0.00 mm, vias 2 -> 0
- net SLOT_WAIT: track 52.4 -> 0.00 mm, vias 2 -> 0
- net UART_RX: track 45.7 -> 0.00 mm, vias 1 -> 0
- net SLOT_RESET_N: track 45.3 -> 0.00 mm, vias 2 -> 0
- net D7: track 44.7 -> 0.00 mm, vias 1 -> 0
- net SLOT_WR_N: track 44.6 -> 0.00 mm, vias 2 -> 0
- net SLOT_RD_N: track 44.4 -> 0.00 mm, vias 2 -> 0
- net UART_TX: track 43.8 -> 0.00 mm, vias 1 -> 0
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- removed copper zone on B.Cu, net GND
- removed copper zone on F.Cu, net GND
Other:
- board size 95.2 x 65.4 mm -> 95 x 95 mm
- board text removed: "(C)2026 HRA!"
- board text removed: "3V3"
- board text removed: "BCLK"
- board text removed: "GND"
- board text removed: "JTAG"
- board text removed: "LRCLK"
- board text removed: "MCLK"
- board text removed: "OFF"
- board text removed: "ON"
- board text removed: "Prototype Rev.1"
- board text removed: "ROM"
- board text removed: "SDAT"
- board text removed: "SNDIN"
- board text removed: "TangPrimer25K"
- board text removed: "Y8960 Cartridge"
