File: pcb/FPGA_MSXtR_Stack_CPU/StackCPU.kicad_sch (KiCad schematic)
At the start: 34 parts, among them J1 MSX_EXBUS_A, J2 MSX_EXBUS_B, J3 I2S_CONN, J4 Conn_02x06_Odd_Even, J5 GND, J6 SOUNDIN

Commit message: Updated
Parts:
- U1: footprint My Parts:TangPrimer25K(UPPER) -> 0-My_Parts:TangPrimer25K(UPPER)
- U3: renamed from U4; footprint My Parts:CLOCK -> 0-My_Parts:CLOCK
- U8: renamed from U3; footprint My Parts:QSPI-SRAM 4Mbit (8SOIC) -> 0-My_Parts:QSPI-SRAM 4Mbit (8SOIC)
- U9: renamed from U2; footprint My Parts:TangPrimer25K(LOWER) -> 0-My_Parts:TangPrimer25K(LOWER)
- renumbered C2 to C1, C4 to C13, C3 to C2, C1 to C3, J3 to J1, J6 to J2, J4 to J3, J5 to J4, J2 to J5, J1 to J6
Connections:
- net +5V: no longer C13.1, J5.39 (Pin_39), J6.34 (Pin_34)
- net GND: no longer J5.37 (Pin_37), J5.40 (Pin_40), J6.36 (Pin_36)
- net SLOT_INT_N: no longer U9.97 (SLOT_INTR)
- net SLOT_SLTSL0_N: no longer U9.66 (SLOT_SLTSL_N)
- net SLOT_SNDIN: no longer J2.1 (Pin_1)
- net SLOT_WAIT_N: no longer U9.99 (SLOT_WAIT)
- net SLOT_BUSDIR: now reaches U9.103 (SLOT_BUSDIR)
- new net 5V: C13.1, J5.39 (Pin_39), J6.34 (Pin_34)
- new net SLOT_GND: J5.37 (Pin_37), J5.40 (Pin_40), J6.36 (Pin_36)
- new net SLOT_INTR: U9.97 (SLOT_INTR)
- new net SLOT_SLTSL_N: U9.66 (SLOT_SLTSL_N)
- new net SLOT_WAIT: U9.99 (SLOT_WAIT)
- no-connect marks 51 -> 38
Other:
- moved on the sheet: C1, C13, C2, C3, J1, J2, J3, J4, J5, J6, SW1, SW2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

Commit message: Updated
Parts:
- removed D1, D2, D3, D4: LED, LED_SMD:LED_0805_2012Metric, symbol Device:LED
- removed J1: I2S_CONN, Connector_PinHeader_2.54mm:PinHeader_1x06_P2.54mm_Vertical, symbol Connector_Generic:Conn_01x06
- removed J2: SOUNDIN, Connector_PinHeader_2.54mm:PinHeader_1x01_P2.54mm_Vertical, symbol Connector_Generic:Conn_01x01
- removed J4: GND, Connector_PinHeader_2.54mm:PinHeader_1x01_P2.54mm_Vertical, symbol Connector_Generic:Conn_01x01
- removed R10, R11, R12, R9: 3.3k, Resistor_SMD:R_0805_2012Metric, symbol Device:R
- removed R24, R25, R26, R27: 470, Resistor_SMD:R_0805_2012Metric, symbol Device:R
- removed SW1, SW2: ~, 0-My_Parts:SlideSW_Side, symbol My Parts:Switch
- added C10, C11, C4, C5, C6, C9: 0.1uF, Capacitor_SMD:C_0402_1005Metric, symbol Device:C
- added C8: 1uF, Capacitor_SMD:C_0402_1005Metric, symbol Device:C
- added J4: Micro_SD_Card, 0-My_Parts:MicroSD(C91145), symbol Connector:Micro_SD_Card
- added J5: Keybard I2C Connector, 0-My_Parts:Grove_I2C, symbol Connector:Conn_01x04_Pin
- added J6: USB_C_Receptacle_PowerOnly_6P, 0-My_Parts:USB-C(C2927029), symbol Connector:USB_C_Receptacle_PowerOnly_6P
- added R1, R2: 5.1K, Resistor_SMD:R_0603_1608Metric, symbol Device:R
- added R13, R14: 100K, Resistor_SMD:R_0402_1005Metric, symbol Device:R
- added R3, R4, R5, R6: 22K, Resistor_SMD:R_0402_1005Metric, symbol Device:R
- added SW1: SW_MEC_5G, symbol Switch:SW_MEC_5G
- added SW3: SW_DIP_x04, symbol Switch:SW_DIP_x04
- added U10: W25Q32JVSS, Package_SO:SOIC-8_5.3x5.3mm_P1.27mm, symbol Memory_Flash:W25Q32JVSS
- added U11, U12: ~, symbol My Parts:FlashROM(8bit)_4Mbit
- added U4: ~, symbol My Parts:FPGA_MSXtR_PICO
- added U6, U7, U8: ~, My Parts:QSPI-SRAM 4Mbit (8SOIC), symbol My Parts:QSPI-SRAM_4Mbit
- added U9: ~, symbol My Parts:DCDC12V_MAU108
- U1: footprint 0-My_Parts:TangPrimer25K(UPPER) -> My Parts:TangPrimer25K(UPPER); symbol My Parts:Y8960(UPPER) -> My Parts:FPGA_MSX_CPU(UPPER)
- U2: renamed from U9; footprint 0-My_Parts:TangPrimer25K(LOWER) -> My Parts:TangPrimer25K(LOWER); symbol My Parts:Y8960(LOWER) -> My Parts:FPGA_MSX_CPU(LOWER)
- U3: footprint 0-My_Parts:CLOCK -> My Parts:CLOCK
- U5: renamed from U8; footprint 0-My_Parts:QSPI-SRAM 4Mbit (8SOIC) -> My Parts:QSPI-SRAM 4Mbit (8SOIC)
- renumbered C13 to C7, J6 to J1, J5 to J2, R15 to R10, R17 to R11, R18 to R12, R16 to R7, R14 to R8, R13 to R9
Connections:
- net 3V3 is gone; now on net +3V3: J2.35 (Pin_35)
- net 5V is gone; now on net +5V: C7.1, J1.34 (Pin_34), J2.39 (Pin_39)
- net SLOT_BUSDIR is gone; now on net SLOT_BUSDIR_N: U2.103 (SLOT_BUSDIR_N)
- net SLOT_GND is gone; now on net GND: J1.36 (Pin_36), J2.37 (Pin_37), J2.40 (Pin_40)
- net SLOT_INTR is gone; now on net SLOT_INT_N: U2.97 (SLOT_INT_N)
- net SLOT_SLTSL_N is gone; now on net SLOT_RFSH_N: U2.66 (SLOT_RFSH_N)
- net SLOT_WAIT is gone; now on net SLOT_WAIT_N: U2.99 (SLOT_WAIT_N)
- net +12V: now also R13.2, U9.6 (+12V)
- net +3V3: now also C10.1, C11.1, C4.1, C5.1, C6.1, C9.2, J4.4 (VDD), J5.3 (Pin_3), R3.2, R4.2, R5.2, R6.2, U10.3 (~{WP}/IO_{2}), U10.7 (~{HOLD}/~{RESET}/IO_{3}), U10.8 (VCC), U11.8 (VCC), U12.8 (VCC), U6.8 (VCC), U7.8 (VCC), U8.8 (VCC)
- net +5V: now also C8.1, J6.A9 (VBUS), J6.B9 (VBUS), U4.40 (VBUS), U9.1 (+5V)
- net -12V: now also R14.1, U9.4 (-12V)
- net DIPSW0: now also SW3.1, U4.25 (GP19); no longer U2.77 (DIPSW0(READY))
- net DIPSW1: now also SW3.2, U4.24 (GP18); no longer U2.83 (DIPSW1)
- net GND: now also C10.2, C11.2, C4.2, C5.2, C6.2, C8.2, C9.1, J4.6 (VSS), J5.4 (Pin_4), J6.A12 (GND), J6.B12 (GND), R1.2, R13.1, R14.2, R2.2, SW1.3 (B), SW1.4 (B), SW3.5, SW3.6, SW3.7, SW3.8, U10.4 (GND), U11.24 (GND), U12.24 (GND), U4.13 (GND), U4.18 (GND), U4.23 (GND), U4.28 (GND), U4.33 (GND), U4.38 (GND), U4.8 (GND), U6.4 (VSS), U7.4 (VSS), U8.4 (VSS), U9.2 (GND), U9.5 (COMMON)
- net SLOT_A0: now also U11.20 (A0), U12.20 (A0)
- net SLOT_A1: now also U11.19 (A1), U12.19 (A1)
- net SLOT_A10: now also U11.31 (A10), U12.31 (A10)
- net SLOT_A11: now also U11.1 (A11), U12.1 (A11)
- net SLOT_A12: now also U11.12 (A12), U12.12 (A12)
- net SLOT_A13: now also U11.4 (A13), U12.4 (A13)
- net SLOT_A14: now also U11.5 (A14), U12.5 (A14)
- net SLOT_A15: now also U11.11 (A15), U12.11 (A15)
- net SLOT_A2: now also U11.18 (A2), U12.18 (A2)
- net SLOT_A3: now also U11.17 (A3), U12.17 (A3)
- net SLOT_A4: now also U11.16 (A4), U12.16 (A4)
- net SLOT_A5: now also U11.15 (A5), U12.15 (A5)
- net SLOT_A6: now also U11.14 (A6), U12.14 (A6)
- net SLOT_A7: now also U11.13 (A7), U12.13 (A7)
- net SLOT_A8: now also U11.3 (A8), U12.3 (A8)
- net SLOT_A9: now also U11.2 (A9), U12.2 (A9)
- net SLOT_CLOCK_N: now also U2.77 (SLOT_CLOCK_N(READY))
- net SLOT_CS12_N: now also U2.85 (SLOT_CS12_N(DONE))
- net SLOT_CS1_N: now also U1.10 (SLOT_CS1_N)
- net SLOT_CS2_N: now also U1.12 (SLOT_CS2_N)
- net SLOT_D0: now also U11.21 (D0), U12.21 (D0)
- net SLOT_D1: now also U11.22 (D1), U12.22 (D1)
- net SLOT_D2: now also U11.23 (D2), U12.23 (D2)
- net SLOT_D3: now also U11.25 (D3), U12.25 (D3)
- net SLOT_D4: now also U11.26 (D4), U12.26 (D4)
- net SLOT_D5: now also U11.27 (D5), U12.27 (D5)
- net SLOT_D6: now also U11.28 (D6), U12.28 (D6)
- net SLOT_D7: now also U11.29 (D7), U12.29 (D7)
- net SLOT_M1_N: now also U1.3 (SLOT_M1_N); no longer U1.6 (SLOT_M1_N)
- net SLOT_RD_N: now also U11.32 (/OE), U12.32 (/OE)
- net SLOT_SLTSL0_N: now also U1.30 (SLOT_SLTSL0_N)
- net SLOT_SLTSL1_N: now also U1.32 (SLOT_SLTSL1_N)
- net SLOT_SLTSL2_N: now also U1.34 (SLOT_SLTSL2_N)
- net SLOT_SLTSL3_N: now also U1.36 (SLOT_SLTSL3_N)
- net SLOT_WR_N: now also U11.7 (/WE), U12.7 (/WE)
- net SRAM_SCLK: now also U6.6 (SCK), U7.6 (SCK), U8.6 (SCK)
- net SRAM_SIO0: now also R9.2, U1.9 (SRAM_SIO0), U6.5 (SI/SIO0), U7.5 (SI/SIO0), U8.5 (SI/SIO0); no longer R10.2, U1.11 (SRAM_SIO0)
- net SRAM_SIO1: now also R10.2, U1.11 (SRAM_SIO1), U6.2 (SO/SIO1), U7.2 (SO/SIO1), U8.2 (SO/SIO1); no longer R7.2, U1.5 (SRAM_SIO1)
- net SRAM_SIO2: now also U6.3 (SIO2), U7.3 (SIO2), U8.3 (SIO2)
- net SRAM_SIO3: now also U6.7 (~{HOLD}/SIO3), U7.7 (~{HOLD}/SIO3), U8.7 (~{HOLD}/SIO3)
- net SLOT_A16: now reaches U2.111 (SLOT_A16)
- net SLOT_A16: now also U11.10 (A16), U12.10 (A16)
- net SLOT_A17: now reaches U2.113 (SLOT_A17)
- net SLOT_A17: now also U11.6 (A17), U12.6 (A17)
- net SLOT_A18: now reaches U2.115 (SLOT_A18)
- net SLOT_A18: now also U11.9 (A18), U12.9 (A18)
- net SLOT_ROM1_CE_N: now reaches U2.117 (SLOT_ROM1_CE_N)
- net SLOT_ROM1_CE_N: now also U12.30 (/CE)
- net SLOT_DATA_DIR: now reaches J2.5 (Pin_5)
- net SLOT_DATA_DIR: now also U1.6 (SLOT_DATA_DIR)
- net SLOT_OE_N: now reaches J2.7 (Pin_7)
- net SLOT_OE_N: now also R7.2, U1.5 (SLOT_OE_N)
- net MCU_CS_N: now reaches U1.14 (MCU_CS_N)
- net MCU_CS_N: now also U4.7 (FPGA_SPI_CS_N(GP5))
- net MCU_SCLK: now reaches U1.16 (MCU_SCLK)
- net MCU_SCLK: now also U4.9 (FPGA_SPI_CLK(GP6))
- net MCU_MOSI: now reaches U1.18 (MCU_MOSI)
- net MCU_MOSI: now also U4.10 (FPGA_SPI_MOSI(GP7))
- net MCU_MISO: now reaches U1.20 (MCU_MISO)
- net MCU_MISO: now also U4.6 (FPGA_SPI_MISO(GP4))
- net SRAM_CS0_N: now reaches U1.22 (SRAM_CS0_N)
- net SRAM_CS0_N: now also U5.1 (~{CS})
- net SRAM_CS1_N: now reaches U1.24 (SRAM_CS1_N)
- net SRAM_CS1_N: now also U6.1 (~{CS})
- net SRAM_CS2_N: now reaches U1.26 (SRAM_CS2_N)
- net SRAM_CS2_N: now also U7.1 (~{CS})
- net SRAM_CS3_N: now reaches U1.28 (SRAM_CS3_N)
- net SRAM_CS3_N: now also U8.1 (~{CS})
- net SLOT_ROM0_CE_N: now reaches U1.8 (SLOT_ROM0_CE_N)
- net SLOT_ROM0_CE_N: now also U11.30 (/CE)
- net AUDIO_BCLK renamed SROM_CS_N
- net SROM_CS_N: now also U10.1 (~{CS})
- net AUDIO_LRCLK renamed SROM_MOSI
- net SROM_MOSI: now also U10.5 (DI/IO_{0})
- net AUDIO_MCLK renamed SROM_SCLK
- net SROM_SCLK: now also U10.6 (CLK)
- net AUDIO_SDATA renamed SROM_MISO
- net SROM_MISO: now also U10.2 (DO/IO_{1})
- net SLOT_SNDIN: no longer names the net of J2.1 (Pin_1)
- removed net SRAM_CS_N: R9.2, U1.9 (SRAM_CS_N), U5.1 (~{CS})
- new net: J6.A5 (CC1), R1.1
- new net: J6.B5 (CC2), R2.1
- new net DIPSW2: SW3.3, U4.22 (GP17)
- new net DIPSW3: SW3.4, U4.21 (GP16)
- new net I2C_SCL: J5.2 (Pin_2), U4.27 (GP21)
- new net I2C_SDA: J5.1 (Pin_1), U4.26 (GP20)
- new net MCU_INTR: U2.83 (MCU_INTR), U4.5 (FPGA_SPI_INTR(GP3))
- new net RESET_BUTTON: SW1.1 (A), SW1.2 (A), U4.29 (GP22)
- new net SD_SPI_CS_N: J4.2 (DAT3/CD), R3.1, U4.12 (SD_SPI_CS_N(GP9))
- new net SD_SPI_MISO: J4.7 (DAT0), R6.1, U4.11 (SD_SPI_MISO(GP8))
- new net SD_SPI_MOSI: J4.3 (CMD), R4.1, U4.15 (SD_SPI_MOSI(GP11))
- new net SD_SPI_SCK: J4.5 (CLK), R5.1, U4.14 (SD_SPI_SCK(GP10))
- no-connect marks 38 -> 55
Other:
- note added: "DAT0(DO) - MISO CMD(DI) - MOSI"
- note added: "LCSC Part# C129043 x4 switch"
- note added: "LCSC Part# C1525 0.1uF"
- note added: "LCSC Part# C2901579 CLOCK 28.63636MHz"
- note added: "LCSC Part# C63339 15pF"
- note added: "LCSC Part#C19941161 Flash ROM 4Mbit"
- note added: "LCSC Part#C2906286 Side Tactile Button"
- note added: "LCSC Part#C91145 Micro SD Card Slot"
- note added: "SLOT_SNDIN"
- note added: "System ROM (BIOS/DOS/Kanji)"
- note added: "https://akizukidenshi.com/catalog/g/g104134/ DCDC±12V MAU108"
- title: Y8960 Cartridge -> FPGA MSXtR Stack CPU Board
- moved on the sheet: C1, C2, C3, C7, J1, J2, R10, R7, R8, R9, U3, U5

Commit message: Updated
Parts:
- added C12: 470uF, My Parts:Capacitor(C453487), symbol Device:C_Polarized
- added C13: 0.1uF, Capacitor_SMD:C_0402_1005Metric, symbol Device:C
- added R15, R16, R17, R18, R19, R20, R21, R22: 3.3K, Resistor_SMD:R_0402_1005Metric, symbol Device:R
- added SW2: SW_SPDT, My Parts:Slide SW(C7431058), symbol Switch:SW_SPDT
- R10, R11, R12, R7, R8, R9: value 4.7k -> 3.3K; footprint Resistor_SMD:R_0805_2012Metric -> Resistor_SMD:R_0402_1005Metric
- SW1: footprint (none) -> My Parts:SideSW (C2906286)
- U11, U12: footprint (none) -> Package_SO:TSOP-I-32_18.4x8mm_P0.5mm
- U4: footprint (none) -> MCU_RaspberryPi_and_Boards:RPi_Pico_SMD_TH
- U9: footprint (none) -> My Parts:DCDC_MAU108
Connections:
- net +3V3: now also C13.1, R15.2, R16.2, R17.2, R18.2, R19.2, R20.2, R21.2, R22.2
- net +5V: now also C12.1, SW2.2 (B); no longer J6.A9 (VBUS), J6.B9 (VBUS)
- net GND: now also C12.2, C13.2
- net SRAM_CS0_N: now also R15.1
- net SRAM_CS1_N: now also R16.1
- net SRAM_CS2_N: now also R17.1
- net SRAM_CS3_N: now also R18.1
- net SROM_CS_N: now also R20.1
- net SROM_MISO: now also R22.1
- net SROM_MOSI: now also R21.1
- net SROM_SCLK: now also R19.1
- new net: J6.A9 (VBUS), J6.B9 (VBUS), SW2.1 (A)
- no-connect marks 55 -> 56
Other:
- note added: "LCSC Part#C27585175 SystemRAM"
- note added: "LCSC Part#C2927029 USB-C Connector"
- note added: "LCSC Part#C453487 C"
- note added: "LCSC Part#C7431058 Slide SW"
- note added: "LCSC Part#C82344 Extended ROM"
- note added: "POWER SW"
- note removed: "System ROM (BIOS/DOS/Kanji)"

Commit message: Updated
Parts:
- SW3: footprint (none) -> My Parts:DipSW4(C129043)
- U4: footprint MCU_RaspberryPi_and_Boards:RPi_Pico_SMD_TH -> My Parts:RaspberryPiPico2W
Changed lines of the file:
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@@
 	(wire
 		(pts
-			(xy 393.7 31.75) (xy 391.16 31.75)
+			(xy 394.97 31.75) (xy 391.16 31.75)
 		)
 		(stroke
@@
 	(wire
 		(pts
+			(xy 377.19 31.75) (xy 381 31.75)
+		)
+		(stroke
+			(width 0)
+			(type default)
+		)
+	)
+	(wire
+		(pts
 			(xy 245.11 208.28) (xy 245.11 213.36)
 		)
@@
 	(wire
 		(pts
-			(xy 393.7 35.56) (xy 393.7 31.75)
+			(xy 394.97 35.56) (xy 394.97 31.75)
 		)
 		(stroke
@@
 	(global_label "RESET_BUTTON"
 		(shape output)
-		(at 381 31.75 180)
+		(at 377.19 31.75 180)
 		(fields_autoplaced yes)
 		(effects
@@
 		)
 		(property "Intersheetrefs" "${INTERSHEET_REFS}"
-			(at 364.1054 31.75 0)
+			(at 360.2954 31.75 0)
 			(effects
 				(font
@@
 			)
 		)
-		(property "Footprint" ""
+		(property "Footprint" "My Parts:DipSW4(C129043)"
 			(at 309.88 36.83 0)
 			(effects
@@
 			)
 		)
-		(property "Footprint" "MCU_RaspberryPi_and_Boards:RPi_Pico_SMD_TH"
+		(property "Footprint" "My Parts:RaspberryPiPico2W"
 			(at 238.76 58.42 0)
 			(effects
@@
 	(symbol
 		(lib_id "power:GND")
-		(at 393.7 35.56 0)
+		(at 394.97 35.56 0)
 		(unit 1)
 		(exclude_from_sim no)
@@
 		(fields_autoplaced yes)
 		(property "Reference" "#PWR09"
-			(at 393.7 41.91 0)
+			(at 394.97 41.91 0)
 			(effects
 				(font
@@
 		)
 		(property "Value" "GND"
-			(at 393.7 40.64 0)
+			(at 394.97 40.64 0)
 			(effects
 				(font
@@
 		)
 		(property "Footprint" ""
-			(at 393.7 35.56 0)
+			(at 394.97 35.56 0)
 			(effects
 				(font
@@
 		)
 		(property "Datasheet" ""
-			(at 393.7 35.56 0)
+			(at 394.97 35.56 0)
 			(effects
 				(font
@@
 		)
 		(property "Description" "Power symbol creates a global label with name \"GND\" , ground"
-			(at 393.7 35.56 0)
+			(at 394.97 35.56 0)
 			(effects
 				(font

Commit message: Updated
Parts:
- SW1: footprint My Parts:SideSW (C2906286) -> My Parts:SideSW(C963235); LCSC (none) -> C963235
- SW2: LCSC (none) -> C7431058
- SW3: LCSC (none) -> C129043
- U11, U12: footprint Package_SO:TSOP-I-32_18.4x8mm_P0.5mm -> Package_SO:TSOP-I-32_11.8x8mm_P0.5mm
Other:
- note added: "LCSC Part#C43651917 Flash ROM 4Mbit SST39VF040-70"
- note added: "LCSC Part#C963235 Side Tactile Button"
- note removed: "LCSC Part#C2906286 Side Tactile Button"
